Commit message: add wrist_r_link.dae

File: seed_r7_description/urdf/typeG_upperbody/noid_upper_typeg.urdf.xacro (robot description, xacro)
@@ -219,4 +219,24 @@
   </link>
   <xacro:gazebo_link_reference link_name="l_wrist_center" />
+  <link name="l_wrist_r_link">
+    <xacro:unless value="${disable_mesh}"> <visual>
+      <origin xyz="0 0 0" rpy="0 0 0"/>
+      <geometry>
+        <mesh filename="package://seed_r7_description/meshes/typeG_upperbody/l_wrist_r_link.dae" scale="1 1 1" />
+      </geometry>
+    </visual> </xacro:unless>
+    <xacro:unless value="${disable_mesh}"> <collision>
+      <origin xyz="0 0 0" rpy="0 0 0"/>
+      <geometry>
+        <mesh filename="package://seed_r7_description/meshes/typeG_upperbody/l_wrist_r_link.dae" scale="1 1 1" />
+      </geometry>
+    </collision> </xacro:unless>
+    <inertial>
+      <mass value="0.05" />
+      <origin xyz="0 0 0" rpy="0 -0 0"/>
+      <inertia ixx="0.0001" ixy="0" ixz="0" iyy="0.0001" iyz="0" izz="0.0001"/>
+    </inertial>
+  </link>
+  <xacro:gazebo_link_reference link_name="l_wrist_r_link" />
   <link name="neck_link">
     <xacro:unless value="${disable_mesh}"> <visual>
@@ -410,4 +430,24 @@
   </link>
   <xacro:gazebo_link_reference link_name="r_wrist_center" />
+  <link name="r_wrist_r_link">
+    <xacro:unless value="${disable_mesh}"> <visual>
+      <origin xyz="0 0 0" rpy="0 0 0"/>
+      <geometry>
+        <mesh filename="package://seed_r7_description/meshes/typeG_upperbody/r_wrist_r_link.dae" scale="1 1 1" />
+      </geometry>
+    </visual> </xacro:unless>
+    <xacro:unless value="${disable_mesh}"> <collision>
+      <origin xyz="0 0 0" rpy="0 0 0"/>
+      <geometry>
+        <mesh filename="package://seed_r7_description/meshes/typeG_upperbody/r_wrist_r_link.dae" scale="1 1 1" />
+      </geometry>
+    </collision> </xacro:unless>
+    <inertial>
+      <mass value="0.05" />
+      <origin xyz="0 0 0" rpy="0 -0 0"/>
+      <inertia ixx="0.0001" ixy="0" ixz="0" iyy="0.0001" iyz="0" izz="0.0001"/>
+    </inertial>
+  </link>
+  <xacro:gazebo_link_reference link_name="r_wrist_r_link" />
   <joint name="waist_y_joint" type="revolute">
     <parent link="${base_link}"/>
@@ -503,6 +543,6 @@
   <joint name="l_wrist_r_joint" type="revolute">
     <parent link="l_wrist_center"/>
-    <child  link="${l_hand_link}"/>
-    <origin xyz="0 0 0" rpy="0 0 0 "/>
+    <child  link="l_wrist_r_link"/>
+    <origin xyz="0 0 0" rpy="0 -0 0 "/>
     <axis   xyz="1 0 0"/>
     <!-- from -90 to 20 degrees-->
@@ -510,5 +550,11 @@
     <dynamics damping="0.2" friction="0" />
   </joint>
-  <xacro:gazebo_transmission joint_name="l_wrist_r_joint" />
+  <xacro:gazebo_transmission joint_name="r_wrist_r_joint" />
+  <joint name="l_wrist_to_hand_connector" type="fixed">
+    <parent link="l_wrist_r_link"/>
+    <child  link="${l_hand_link}"/>
+    <origin xyz="0 0 -0.004" rpy="0 0 0 "/>
+  </joint>
+  <xacro:gazebo_transmission joint_name="r_wrist_r_joint" />
   <joint name="neck_y_joint" type="revolute">
     <parent link="body_link"/>
@@ -603,5 +649,5 @@
   <joint name="r_wrist_r_joint" type="revolute">
     <parent link="r_wrist_center"/>
-    <child  link="${r_hand_link}"/>
+    <child  link="r_wrist_r_link"/>
     <origin xyz="0 0 0" rpy="0 -0 0 "/>
     <axis   xyz="1 0 0"/>
@@ -611,4 +657,10 @@
   </joint>
   <xacro:gazebo_transmission joint_name="r_wrist_r_joint" />
+  <joint name="r_wrist_to_hand_connector" type="fixed">
+    <parent link="r_wrist_r_link"/>
+    <child  link="${r_hand_link}"/>
+    <origin xyz="0 0 -0.004" rpy="0 0 0 "/>
+  </joint>
+  <xacro:gazebo_transmission joint_name="r_wrist_r_joint" />
   </xacro:macro>
 </robot>

Commit message: fix angle limit

File: seed_r7_description/urdf/typeG_upperbody/noid_upper_typeg.urdf.xacro (robot description, xacro)
@@ -487,5 +487,5 @@
     <!-- from -82 to 18 degrees-->
     <!-- <limit lower="-1.535" upper="0.261" effort="200" velocity="0.4" /> -->
-    <limit lower="-1.43" upper="0.31" effort="200" velocity="0.4" /> -->
+    <limit lower="-1.39" upper="0.31" effort="200" velocity="0.4" /> -->
     <dynamics damping="0.2" friction="0" />
   </joint>
@@ -497,5 +497,5 @@
     <axis   xyz="1 0 0"/>
     <!-- from -10 to 90 degrees-->
-    <limit lower="-0.17" upper="1.5707" effort="100" velocity="0.6" />
+    <limit lower="-0.17" upper="1.57" effort="100" velocity="0.57" />
     <dynamics damping="0.2" friction="0" />
   </joint>
@@ -517,5 +517,5 @@
     <axis   xyz="0 1 0"/>
     <!-- from -171 to 0 degrees-->
-    <limit lower="-3.0" upper="0" effort="100" velocity="1.2" />
+    <limit lower="-3.0" upper="0" effort="100" velocity="1.79" />
     <dynamics damping="0.2" friction="0" />
   </joint>
@@ -537,5 +537,5 @@
     <axis   xyz="0 1 0"/>
     <!-- from -8 to 8 degrees-->
-    <limit lower="-0.14" upper="0.14" effort="100" velocity="0.9" />
+    <limit lower="-0.139" upper="0.139" effort="100" velocity="0.9" />
     <dynamics damping="0.2" friction="0" />
   </joint>
@@ -547,5 +547,5 @@
     <axis   xyz="1 0 0"/>
     <!-- from -90 to 20 degrees-->
-    <limit lower="-1.57" upper="0.35" effort="100" velocity="2.1" />
+    <limit lower="-1.51" upper="0.34" effort="100" velocity="1.8" />
     <dynamics damping="0.2" friction="0" />
   </joint>
@@ -573,5 +573,5 @@
     <axis   xyz="0 1 0"/>
     <!-- from -50 to 40 degrees-->
-    <limit lower="-0.87" upper="0.7" effort="100" velocity="2.1" />
+    <limit lower="-0.87" upper="0.69" effort="100" velocity="2.1" />
     <dynamics damping="0.2" friction="0" />
   </joint>
@@ -583,5 +583,5 @@
     <axis   xyz="1 0 0"/>
     <!-- from -20 to 20 degrees-->
-    <limit lower="-0.35" upper="0.35" effort="100" velocity="0.9" />
+    <limit lower="-0.34" upper="0.34" effort="100" velocity="0.8" />
     <dynamics damping="0.2" friction="0" />
   </joint>
@@ -593,5 +593,5 @@
     <axis   xyz="0 0.984808 0.173648"/>
     <!-- from -82 to 18 degrees-->
-    <limit lower="-1.43" upper="0.31" effort="200" velocity="0.4" /> -->
+    <limit lower="-1.39" upper="0.31" effort="200" velocity="0.4" /> -->
     <dynamics damping="0.2" friction="0" />
   </joint>
@@ -603,5 +603,5 @@
     <axis   xyz="1 0 0"/>
     <!-- from -90 to 10 degrees-->
-    <limit lower="-1.5707" upper="0.17" effort="100" velocity="0.6" />
+    <limit lower="-1.5707" upper="0.17" effort="100" velocity="0.57" />
     <dynamics damping="0.2" friction="0" />
   </joint>
@@ -623,5 +623,5 @@
     <axis   xyz="0 1 0"/>
     <!-- from -171 to 0 degrees-->
-    <limit lower="-3.0" upper="0" effort="100" velocity="1.2" />
+    <limit lower="-3.0" upper="0" effort="100" velocity="1.79" />
     <dynamics damping="0.2" friction="0" />
   </joint>
@@ -643,5 +643,5 @@
     <axis   xyz="0 1 0"/>
     <!-- from -8 to 8 degrees-->
-    <limit lower="-0.14" upper="0.14" effort="100" velocity="0.9" />
+    <limit lower="-0.139" upper="0.139" effort="100" velocity="0.9" />
     <dynamics damping="0.2" friction="0" />
   </joint>
@@ -653,5 +653,5 @@
     <axis   xyz="1 0 0"/>
     <!-- from -20 to 90 degrees-->
-    <limit lower="-0.35" upper="1.57" effort="100" velocity="2.1" />
+    <limit lower="-0.34" upper="1.51" effort="100" velocity="1.8" />
     <dynamics damping="0.2" friction="0" />
   </joint>

Commit message: update joint velocity limit for fullstep transfer

File: seed_r7_description/urdf/typeG_upperbody/noid_upper_typeg.urdf.xacro (robot description, xacro)
@@ -456,5 +456,5 @@
     <axis   xyz="0 0 1"/>
     <!-- from -120 to 120 degrees-->
-    <limit lower="-2.09" upper="2.09" effort="500" velocity="0.6" />
+    <limit lower="-2.09" upper="2.09" effort="500" velocity="1.7" />
     <dynamics damping="0.2" friction="0" />
   </joint>
@@ -466,5 +466,5 @@
     <axis   xyz="0 1 0"/>
     <!-- from -10 to 46 degrees-->
-    <limit lower="-0.17" upper="0.8" effort="2000" velocity="0.5" />
+    <limit lower="-0.17" upper="0.8" effort="2000" velocity="1.6" />
     <dynamics damping="0.2" friction="0" />
   </joint>
@@ -476,5 +476,5 @@
     <axis   xyz="1 0 0"/>
     <!-- from -7 to 7 degrees-->
-    <limit lower="-0.12" upper="0.12" effort="2000" velocity="0.4" />
+    <limit lower="-0.12" upper="0.12" effort="2000" velocity="1.3" />
     <dynamics damping="0.2" friction="0" />
   </joint>
@@ -487,5 +487,5 @@
     <!-- from -82 to 18 degrees-->
     <!-- <limit lower="-1.535" upper="0.261" effort="200" velocity="0.4" /> -->
-    <limit lower="-1.39" upper="0.31" effort="200" velocity="0.4" /> -->
+    <limit lower="-1.39" upper="0.31" effort="200" velocity="0.6" /> -->
     <dynamics damping="0.2" friction="0" />
   </joint>
@@ -497,5 +497,5 @@
     <axis   xyz="1 0 0"/>
     <!-- from -10 to 90 degrees-->
-    <limit lower="-0.17" upper="1.57" effort="100" velocity="0.57" />
+    <limit lower="-0.17" upper="1.57" effort="100" velocity="1.0" />
     <dynamics damping="0.2" friction="0" />
   </joint>
@@ -507,5 +507,5 @@
     <axis   xyz="0 0 1"/>
     <!-- from -180 to 180 degrees-->
-    <limit lower="-1.5707" upper="1.5707" effort="100" velocity="1.2" />
+    <limit lower="-1.5707" upper="1.5707" effort="100" velocity="1.7" />
     <dynamics damping="0.2" friction="0" />
   </joint>
@@ -517,5 +517,5 @@
     <axis   xyz="0 1 0"/>
     <!-- from -171 to 0 degrees-->
-    <limit lower="-3.0" upper="0" effort="100" velocity="1.79" />
+    <limit lower="-3.0" upper="0" effort="100" velocity="4.4" />
     <dynamics damping="0.2" friction="0" />
   </joint>
@@ -527,5 +527,5 @@
     <axis   xyz="0 0 1"/>
     <!-- from -180 to 180 degrees-->
-    <limit lower="-1.5707" upper="1.5707" effort="100" velocity="1.3" />
+    <limit lower="-1.5707" upper="1.5707" effort="100" velocity="1.9" />
     <dynamics damping="0.2" friction="0" />
   </joint>
@@ -537,5 +537,5 @@
     <axis   xyz="0 1 0"/>
     <!-- from -8 to 8 degrees-->
-    <limit lower="-0.139" upper="0.139" effort="100" velocity="0.9" />
+    <limit lower="-0.139" upper="0.139" effort="100" velocity="1.7" />
     <dynamics damping="0.2" friction="0" />
   </joint>
@@ -547,5 +547,5 @@
     <axis   xyz="1 0 0"/>
     <!-- from -90 to 20 degrees-->
-    <limit lower="-1.51" upper="0.34" effort="100" velocity="1.8" />
+    <limit lower="-1.51" upper="0.34" effort="100" velocity="3.4" />
     <dynamics damping="0.2" friction="0" />
   </joint>
@@ -563,5 +563,5 @@
     <axis   xyz="0 0 1"/>
     <!-- from -120 to 120 degrees-->
-    <limit lower="-2.09" upper="2.09" effort="100" velocity="1.6" />
+    <limit lower="-2.09" upper="2.09" effort="100" velocity="1.7" />
     <dynamics damping="0.2" friction="0" />
   </joint>
@@ -573,5 +573,5 @@
     <axis   xyz="0 1 0"/>
     <!-- from -50 to 40 degrees-->
-    <limit lower="-0.87" upper="0.69" effort="100" velocity="2.1" />
+    <limit lower="-0.87" upper="0.69" effort="100" velocity="4.0" />
     <dynamics damping="0.2" friction="0" />
   </joint>
@@ -583,5 +583,5 @@
     <axis   xyz="1 0 0"/>
     <!-- from -20 to 20 degrees-->
-    <limit lower="-0.34" upper="0.34" effort="100" velocity="0.8" />
+    <limit lower="-0.34" upper="0.34" effort="100" velocity="1.6" />
     <dynamics damping="0.2" friction="0" />
   </joint>
@@ -593,5 +593,5 @@
     <axis   xyz="0 0.984808 0.173648"/>
     <!-- from -82 to 18 degrees-->
-    <limit lower="-1.39" upper="0.31" effort="200" velocity="0.4" /> -->
+    <limit lower="-1.39" upper="0.31" effort="200" velocity="0.6" /> -->
     <dynamics damping="0.2" friction="0" />
   </joint>
@@ -603,5 +603,5 @@
     <axis   xyz="1 0 0"/>
     <!-- from -90 to 10 degrees-->
-    <limit lower="-1.5707" upper="0.17" effort="100" velocity="0.57" />
+    <limit lower="-1.5707" upper="0.17" effort="100" velocity="1.0" />
     <dynamics damping="0.2" friction="0" />
   </joint>
@@ -613,5 +613,5 @@
     <axis   xyz="0 0 1"/>
     <!-- from -180 to 180 degrees-->
-    <limit lower="-1.5707" upper="1.5707" effort="100" velocity="1.2" />
+    <limit lower="-1.5707" upper="1.5707" effort="100" velocity="1.7" />
     <dynamics damping="0.2" friction="0" />
   </joint>
@@ -623,5 +623,5 @@
     <axis   xyz="0 1 0"/>
     <!-- from -171 to 0 degrees-->
-    <limit lower="-3.0" upper="0" effort="100" velocity="1.79" />
+    <limit lower="-3.0" upper="0" effort="100" velocity="4.4" />
     <dynamics damping="0.2" friction="0" />
   </joint>
@@ -633,5 +633,5 @@
     <axis   xyz="0 0 1"/>
     <!-- from -180 to 180 degrees-->
-    <limit lower="-1.5707" upper="1.5707" effort="100" velocity="1.3" />
+    <limit lower="-1.5707" upper="1.5707" effort="100" velocity="1.9" />
     <dynamics damping="0.2" friction="0" />
   </joint>
@@ -643,5 +643,5 @@
     <axis   xyz="0 1 0"/>
     <!-- from -8 to 8 degrees-->
-    <limit lower="-0.139" upper="0.139" effort="100" velocity="0.9" />
+    <limit lower="-0.139" upper="0.139" effort="100" velocity="1.7" />
     <dynamics damping="0.2" friction="0" />
   </joint>
@@ -653,5 +653,5 @@
     <axis   xyz="1 0 0"/>
     <!-- from -20 to 90 degrees-->
-    <limit lower="-0.34" upper="1.51" effort="100" velocity="1.8" />
+    <limit lower="-0.34" upper="1.51" effort="100" velocity="3.4" />
     <dynamics damping="0.2" friction="0" />
   </joint>
