Commit message: add front/rear camer tf and change IK solver

File: seed_r7_description/urdf/typeG_wheel/wheels.urdf.xacro (robot description, xacro)
@@ -185,4 +185,40 @@
       <origin xyz="0.308 0 0.0994" rpy="0 0 0"/>
     </joint>
+    <link name="front_camera_base_link"/>
+    <joint name="wheel_base_link_to_front_camera_base_link" type="fixed">
+      <parent  link="wheel_base_link"/>
+      <child link="front_camera_base_link"/>
+      <origin xyz="0.31815 0 0.0165" rpy="0 0 0"/>
+    </joint>
+    <link name="front_camera_link"/>
+    <joint name="front_camera_base_link_to_front_camera_link" type="fixed">
+      <parent  link="front_camera_base_link"/>
+      <child link="front_camera_link"/>
+      <origin xyz="0 0.0175 0.0125" rpy="0 0 0"/>
+    </joint>
+    <link name="front_camera_right_ir_frame"/>
+    <joint name="front_camera_link_to_front_camera_right_ir_link" type="fixed">
+      <parent  link="front_camera_link"/>
+      <child link="front_camera_right_ir_frame"/>
+      <origin xyz="0 -0.05 0" rpy="0 0 0"/>
+    </joint>
+    <link name="rear_camera_base_link"/>
+    <joint name="wheel_base_link_to_rear_camera_base_link" type="fixed">
+      <parent  link="wheel_base_link"/>
+      <child link="rear_camera_base_link"/>
+      <origin xyz="-0.31815 0 0.0165" rpy="0 0 3.1415926538"/>
+    </joint>
+    <link name="rear_camera_link"/>
+    <joint name="rear_camera_base_link_to_rear_camera_link" type="fixed">
+      <parent  link="rear_camera_base_link"/>
+      <child link="rear_camera_link"/>
+      <origin xyz="0 0.0175 0.0125" rpy="0 0 0"/>
+    </joint>
+    <link name="rear_camera_right_ir_frame"/>
+    <joint name="rear_camera_link_to_rear_camera_right_ir_link" type="fixed">
+      <parent  link="rear_camera_link"/>
+      <child link="rear_camera_right_ir_frame"/>
+      <origin xyz="0 -0.05 0" rpy="0 0 0"/>
+    </joint>
   </xacro:macro>
 </robot>
